File: Hardware/Boards/Multi_PowerSupply/Multi_PowerSupply.sch (KiCad schematic (older format))
At the start: 35 parts, among them J1 Input_1, J10 Output, J11 Conn_01x02_Male, J12 Conn_01x02_Male, J13 Conn_01x02_Male, J14 Conn_01x02_Male, J15 Conn_01x02_Male, J2 Input_2, J3 Input_3, J4 Input_4, J5 Conn_01x02_Male, J6 Conn_01x02_Male, J7 Conn_01x02_Male, J8 Conn_01x02_Male, J9 Conn_01x02_Male

Commit message: Add boards schemetics.
Other:
- note added: "Power Input Terminals\n"
- note added: "Power Output Terminal"
- note added: "Power Saving Jumpers"
- moved on the sheet: C1, C2, C3, C4, C5, D1, D2, D3, D4, D5, D6, D7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

Commit message: Add boards and report in tex.
Parts:
- removed D9: LED, _018:LED_D3.0mm, symbol Device:LED
- removed J15, J9: Conn_01x02_Male, Connector_PinHeader_2.54mm:PinHeader_1x02_P2.54mm_Vertical, symbol Connector:Conn_01x02_Male
- removed R5: R, _018:Res_Small, symbol Device:R
- added J16: Conn_01x05, _019:Molex_5, symbol Connector_Generic:Conn_01x05
- added J17: Conn_02x05_Top_Bottom, Connector_PinHeader_2.54mm:PinHeader_2x05_P2.54mm_Vertical, symbol Connector_Generic:Conn_02x05_Odd_Even
- added U1: Buck, _018:Buck_Regulator, symbol custom_symbols:Buck
- J1, J2, J3, J4: footprint _018:bornier2-medium -> _018:Solar_Connector
Connections:
- net labels added: VCC
- wire segments 68 -> 99
- no-connect marks 10 -> 8
Other:
- note added: "Power Output Terminals"
- note removed: "Power Output Terminal"
- moved on the sheet: C5, J10, J11, J12, J13, J14
